File: eagle/v0.2/PaxInstruments-T100.brd (EAGLE design)
At the start: 45.1 x 17.1 mm, 29 parts, among them U1 Attiny85

Commit message: Date code and version number updated
Other:
- board text added: "Pax Instruments T-100 [v0.2] January 2015"
- board text removed: "Pax Instruments T-100 [v0.1] November 2014"
Changed lines of the file:
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@@
 <wire x1="23.1775" y1="7.3025" x2="23.1775" y2="2.8575" width="1.016" layer="46"/>
 <text x="44.45" y="7.3025" size="1.016" layer="26" font="vector" rot="MR0">Pax Instruments T-100
-[v0.1] November 2014</text>
+[v0.2] January 2015</text>
 </plain>
 <attributes>
