File: eagle/v0.2/PaxInstruments-T100.sch (EAGLE design)
At the start: 29 parts, among them U1 Attiny85

Commit message: Date code and version number updated
Other:
- note added: "v0.2"
- note removed: "v0.1"
Changed lines of the file:
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@@
 <wire x1="254" y1="116.84" x2="147.32" y2="116.84" width="0.4064" layer="94"/>
 <wire x1="254" y1="66.04" x2="147.32" y2="66.04" width="0.4064" layer="94"/>
-<text x="248.92" y="5.08" size="2.54" layer="94">v0.1</text>
+<text x="248.92" y="5.08" size="2.54" layer="94">v0.2</text>
 </plain>
 <instances>
