File: eagle/v0.3/PaxInstruments-T100.sch (EAGLE design)
At the start: 32 parts, among them U1 Attiny85

Commit message: Changed USB connector. Updated thermocouple footprint. Rerouted board.
Parts:
- removed JP1: USB-A-H, SparkFun-Connectors:USB-A-H
- removed R11, R12: 0R, rcl:R-EU_R0603
- added JP4: USBA-SMD-MALE, SparkFun-Connectors:USBA-SMD-MALE
- added SJ1, SJ2: JUMPER-PAD-2-NC_BY_TRACENO_SILK, SparkFun-Passives:JUMPER-PAD-2-NC_BY_TRACENO_SILK
Connections:
- net AGND: now also SJ2.2; no longer R11.1
- net A_5V: now also SJ1.1; no longer R12.1
- net GND: now also JP4.VBUS, SJ2.1; no longer JP1.VBUS, R11.2
- net N$1: now also JP4.D+; no longer JP1.D+
- net N$2: now also JP4.D-; no longer JP1.D-
- net USB_5V: now also JP4.GND, SJ1.2; no longer JP1.GND, R12.2
